File: hardware/ps2/ps2usb.kicad_sch (KiCad schematic)
At the start: 19 parts, among them J1 DIN8, J2 DIN8, J3 USB1035, J4 Conn_01x03_Pin, U1 CH559L-less, Y1 12MHz

Commit message: Clean up of labels and logo.
Parts:
- D1: footprint ps2usb:B3173BGR-20C0001Q3U1930 -> HIDmanLibrary:B3173BGR-20C0001Q3U1930
- J1: footprint ps2usb:DIN8 -> HIDmanLibrary:DIN8
Changed lines of the file:
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@@
 			)
 		)
-		(property "Footprint" "ps2usb:DIN8"
+		(property "Footprint" "HIDmanLibrary:DIN8"
 			(at 207.01 88.9 0)
 			(effects
@@
 			)
 		)
-		(property "Footprint" "ps2usb:B3173BGR-20C0001Q3U1930"
+		(property "Footprint" "HIDmanLibrary:B3173BGR-20C0001Q3U1930"
 			(at 179.07 114.3 0)
 			(effects

Commit message: Corrected SMD sizes, updated BOM and placement.
Parts:
- C1, C2, C5, C6, C7: footprint Capacitor_SMD:C_1206_3216Metric -> Capacitor_SMD:C_0603_1608Metric
Changed lines of the file:
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@@
 			)
 		)
-		(property "Footprint" "Capacitor_SMD:C_1206_3216Metric"
+		(property "Footprint" "Capacitor_SMD:C_0603_1608Metric"
 			(at 101.6 90.17 0)
 			(effects
@@
 			)
 		)
-		(property "Footprint" "Capacitor_SMD:C_1206_3216Metric"
+		(property "Footprint" "Capacitor_SMD:C_0603_1608Metric"
 			(at 105.41 90.17 0)
 			(effects
@@
 			)
 		)
-		(property "Footprint" "Capacitor_SMD:C_1206_3216Metric"
+		(property "Footprint" "Capacitor_SMD:C_0603_1608Metric"
 			(at 88.9 121.92 0)
 			(effects
@@
 			)
 		)
-		(property "Footprint" "Capacitor_SMD:C_1206_3216Metric"
+		(property "Footprint" "Capacitor_SMD:C_0603_1608Metric"
 			(at 95.25 121.92 0)
 			(effects
@@
 			)
 		)
-		(property "Footprint" "Capacitor_SMD:C_1206_3216Metric"
+		(property "Footprint" "Capacitor_SMD:C_0603_1608Metric"
 			(at 196.85 81.28 0)
 			(effects
